Commit message: Lesson 5

File: src/my_r2d2/urdf/r2d2.urdf (robot description, URDF)
Before this commit: robot physics, 16 links, 15 joints
Links:
- added link base_footprint
Joints:
- added joint base_footprint: type fixed, parent base_link, child base_footprint, origin xyz=0 0 -0.47

Commit message: Lesson URDF

File: src/my_r2d2/urdf/r2d2.urdf (robot description, URDF)
Before this commit: robot physics, 17 links, 16 joints
Joints:
- joint base_footprint: child base_footprint -> base_link; origin xyz=0 0 -0.47 -> xyz=0 0 0.47; parent base_link -> base_footprint

File: src/my_r2d2/urdf/r2d2.xacro (robot description, xacro)
@@ -1,5 +1,9 @@
-<?xml version="1.0"?>
+<?xml version="1.0" ?>
+<!-- =================================================================================== -->
+<!-- |    This document was autogenerated by xacro from r2d2.urdf                      | -->
+<!-- |    EDITING THIS FILE BY HAND IS NOT RECOMMENDED                                 | -->
+<!-- =================================================================================== -->
 <robot name="physics">
-<material name="blue">
+  <material name="blue">
     <color rgba="0 0 0.8 1"/>
   </material>
@@ -27,9 +31,10 @@
     </inertial>
   </link>
-<link name="base_footprint">
+  <link name="base_footprint">
   </link>
   <joint name="base_footprint" type="fixed">
-    <parent link="base_footprint"/>
-    <child link="base_link"/>
+    <parent link="base_link"/>
+    <child link="base_footprint"/>
+    <origin xyz="0 0 -0.47"/>
   </joint>
   <link name="right_leg">

Commit message: AR tracking

File: src/my_r2d2/urdf/r2d2.urdf (robot description, URDF)
Before this commit: robot physics, 17 links, 16 joints
Links:
- added link eye
Joints:
- added joint eye: type fixed, parent box, child eye, origin xyz=0 0 0 rpy=-1.57075 0 -1.57075
